Commit message: 1.- Modify controller parameters 2.- Modify the absolute routes of the mesh files to relative routes 3.- Add an if to be able to stop controllers

File: alpha_description/xacro/alpha.urdf.xacro (robot description, xacro)
@@ -27,5 +27,5 @@
       <visual>
         <geometry>
-          <mesh filename="file://$(find ${description_package})/meshes/M3-INLINE.stl" />
+          <mesh filename="package://${description_package}/meshes/M3-INLINE.stl" />
         </geometry>
         <origin rpy="0 0 0" xyz="0 0 0" />
@@ -54,5 +54,5 @@
       <visual>
         <geometry>
-          <mesh filename="file://$(find ${description_package})/meshes/M2-1-1.stl" />
+          <mesh filename="package://${description_package}/meshes/M2-1-1.stl" />
         </geometry>
         <origin rpy="0 0 0" xyz="0 0 0" />
@@ -81,5 +81,5 @@
       <visual>
         <geometry>
-          <mesh filename="file://$(find ${description_package})/meshes/M2.stl" />
+          <mesh filename="package://${description_package}/meshes/M2.stl" />
         </geometry>
         <origin rpy="0 0 0" xyz="0 0 0" />
@@ -120,5 +120,5 @@
       <visual>
         <geometry>
-          <mesh filename="file://$(find ${description_package})/meshes/M2-1-3.stl" />
+          <mesh filename="package://${description_package}/meshes/M2-1-3.stl" />
         </geometry>
         <origin rpy="0 0 0" xyz="0 0 0" />
@@ -147,6 +147,5 @@
       <visual>
         <geometry>
-          <mesh
-            filename="file://$(find ${description_package})/meshes/RS1-100-101-123.stl" />
+          <mesh filename="package://${description_package}/meshes/RS1-100-101-123.stl" />
         </geometry>
         <origin rpy="0 -1.5707 0" xyz="0 0 0" />

File: alpha_description/xacro/end_effectors/standard_jaws.urdf.xacro (robot description, xacro)
@@ -9,6 +9,5 @@
       <visual>
         <geometry>
-          <mesh
-            filename="file://$(find ${description_package})/meshes/end_effectors/RS1-124.stl" />
+          <mesh filename="package://${description_package}/meshes/end_effectors/RS1-124.stl" />
         </geometry>
         <material name="${prefix}black" />
@@ -36,6 +35,5 @@
       <visual>
         <geometry>
-          <mesh
-            filename="file://$(find ${description_package})/meshes/end_effectors/RS1-130.stl" />
+          <mesh filename="package://${description_package}/meshes/end_effectors/RS1-130.stl" />
         </geometry>
         <material name="${prefix}black" />
@@ -64,6 +62,5 @@
       <visual>
         <geometry>
-          <mesh
-            filename="file://$(find ${description_package})/meshes/end_effectors/RS1-139.stl" />
+          <mesh filename="package://${description_package}/meshes/end_effectors/RS1-139.stl" />
         </geometry>
         <material name="${prefix}black" />
