Commit message: ajuste de sensor

File: alpha_description/xacro/end_effectors/force_sensor.urdf.xacro (robot description, xacro)
@@ -35,5 +35,5 @@
       <visual>
         <geometry>
-          <mesh filename="package://${description_package}/meshes/end_effectors/force_sensor.stl" />
+          <mesh filename="package://${description_package}/meshes/end_effectors/force_sensor.dae" />
         </geometry>
         <origin xyz="0 0 0.01" rpy="0 0 0"/>
@@ -71,5 +71,5 @@
     </joint>
     <joint name="${prefix}force_sensor_joint" type="fixed">
-      <origin xyz="0 0 0.02" rpy="0 0 0"/>
+      <origin xyz="-0.01 0.0 0.0" rpy="1.57 0.0 1.57"/>
       <parent link="${prefix}tool"/>
       <child link="${prefix}force_sensor_link"/>

Commit message: Ajuste para publicar trasnformada de sensores

File: alpha_description/xacro/end_effectors/force_sensor.urdf.xacro (robot description, xacro)
@@ -32,5 +32,5 @@
       </inertial>
     </link>
-    <link name="${prefix}force_sensor_link">
+    <link name="${prefix}link">
       <visual>
         <geometry>
@@ -59,4 +59,18 @@
       </inertial>
     </link>
+    <link name="${prefix}4N">
+    </link>
+    <link name="${prefix}111N">
+    </link>
+    <joint name="${prefix}4N_joint" type="fixed">
+      <origin xyz="0 0.03 0.0" rpy="1.57 0.0 1.57" />
+      <parent link="${prefix}tool" />
+      <child link="${prefix}4N" />
+    </joint>
+    <joint name="${prefix}111N_joint" type="fixed">
+      <origin xyz="0 -0.03 0.0" rpy="1.57 0.0 1.57" />
+      <parent link="${prefix}tool" />
+      <child link="${prefix}111N" />
+    </joint>
     <joint name="${prefix}base_joint" type="fixed">
       <xacro:insert_block name="origin" />
@@ -73,5 +87,5 @@
       <origin xyz="-0.01 0.0 0.0" rpy="1.57 0.0 1.57"/>
       <parent link="${prefix}tool"/>
-      <child link="${prefix}force_sensor_link"/>
+      <child link="${prefix}link"/>
     </joint>
   </xacro:macro>

Commit message: ajuste de trasnformada sensor de fuerza

File: alpha_description/xacro/end_effectors/force_sensor.urdf.xacro (robot description, xacro)
@@ -64,10 +64,10 @@
     </link>
     <joint name="${prefix}4N_joint" type="fixed">
-      <origin xyz="0 0.03 0.0" rpy="1.57 0.0 1.57" />
+      <origin xyz="0 -0.03 0.0" rpy="1.57 0.0 1.57" />
       <parent link="${prefix}tool" />
       <child link="${prefix}4N" />
     </joint>
     <joint name="${prefix}111N_joint" type="fixed">
-      <origin xyz="0 -0.03 0.0" rpy="1.57 0.0 1.57" />
+      <origin xyz="0 0.03 0.0" rpy="1.57 0.0 1.57" />
       <parent link="${prefix}tool" />
       <child link="${prefix}111N" />
